Commit message: added gripper and ball to move to

File: coppelia/GEN3-LITE.urdf (robot description, URDF)
Before this commit: robot KR7108-URDF, 8 links, 7 joints
Links:
- link ARM: geometry collision mesh filename=/home/abban/b38ro-project/kortex_description/gen3_lite/ARM.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; visual mesh filename=/home/abban/b38ro-project/kortex_description/gen3_lite/ARM.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
- link BASE: geometry collision mesh filename=/home/abban/b38ro-project/kortex_description/gen3_lite/BASE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; visual mesh filename=/home/abban/b38ro-project/kortex_description/gen3_lite/BASE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
- link FOREARM: geometry collision mesh filename=/home/abban/b38ro-project/kortex_description/gen3_lite/FORE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; visual mesh filename=/home/abban/b38ro-project/kortex_description/gen3_lite/FORE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
- link LOWER_WRIST: geometry collision mesh filename=/home/abban/b38ro-project/kortex_description/gen3_lite/LOWE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; visual mesh filename=/home/abban/b38ro-project/kortex_description/gen3_lite/LOWE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
- link SHOULDER: geometry collision mesh filename=/home/abban/b38ro-project/kortex_description/gen3_lite/SHOU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; visual mesh filename=/home/abban/b38ro-project/kortex_description/gen3_lite/SHOU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
- link UPPER_WRIST: geometry collision mesh filename=/home/abban/b38ro-project/kortex_description/gen3_lite/UPPE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; visual mesh filename=/home/abban/b38ro-project/kortex_description/gen3_lite/UPPE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
